File: pcb/zx-spectrum-diagnostics.kicad_pcb (KiCad board)
At the start: 2 copper layers, 99.9 x 98.2 mm, 74 parts, among them J101 Conn_01x04, J201 Conn_01x20_Female, J202 Conn_01x20_Female, J203 Conn_01x20_Female, Q101 PMBT2222A, SW101 SW_SPST, U101 Pico, U102 Pico

Commit message: update v1.2 pcb, add comments to PGS version, create v1.2 gerbers
Changed lines of the file:
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@@
       (drillshape 0)
       (scaleselection 1)
-      (outputdirectory "./fab1.1")
+      (outputdirectory "./fab1.2")
     )
   )
@@
     (fp_line (start -1.2 0.8) (end -1.6 0.4) (layer "B.Fab") (width 0.1))
     (fp_line (start -1.6 -0.8) (end 1.6 -0.8) (layer "B.Fab") (width 0.1))
-    (pad "1" smd roundrect (at -1.4875 0 180) (size 1.425 1.75) (layers "B.Cu" "B.Paste" "B.Mask") (roundrect_rratio 0.175439)
+    (pad "1" smd roundrect (at -1.4875 0 180) (size 1.425 1.75) (layers "B.Cu" "B.Paste" "B.Mask") (roundrect_rratio 0.1754392982)
       (net 3 "3V3_PICO1") (pinfunction "K") (pintype "passive"))
-    (pad "2" smd roundrect (at 1.4875 0 180) (size 1.425 1.75) (layers "B.Cu" "B.Paste" "B.Mask") (roundrect_rratio 0.175439)
+    (pad "2" smd roundrect (at 1.4875 0 180) (size 1.425 1.75) (layers "B.Cu" "B.Paste" "B.Mask") (roundrect_rratio 0.1754392982)
       (net 4 "MIN5V_DIV") (pinfunction "A") (pintype "passive"))
     (model "${KICAD6_3DMODEL_DIR}/Diode_SMD.3dshapes/D_1206_3216Metric.wrl"
@@
     (fp_line (start 1.6 -0.8) (end 1.6 0.8) (layer "B.Fab") (width 0.1))
     (fp_line (start -1.6 -0.8) (end 1.6 -0.8) (layer "B.Fab") (width 0.1))
-    (pad "1" smd roundrect (at -1.4875 0 180) (size 1.425 1.75) (layers "B.Cu" "B.Paste" "B.Mask") (roundrect_rratio 0.175439)
+    (pad "1" smd roundrect (at -1.4875 0 180) (size 1.425 1.75) (layers "B.Cu" "B.Paste" "B.Mask") (roundrect_rratio 0.1754392982)
       (net 4 "MIN5V_DIV") (pinfunction "K") (pintype "passive"))
-    (pad "2" smd roundrect (at 1.4875 0 180) (size 1.425 1.75) (layers "B.Cu" "B.Paste" "B.Mask") (roundrect_rratio 0.175439)
+    (pad "2" smd roundrect (at 1.4875 0 180) (size 1.425 1.75) (layers "B.Cu" "B.Paste" "B.Mask") (roundrect_rratio 0.1754392982)
       (net 5 "GND") (pinfunction "A") (pintype "passive"))
     (model "${KICAD6_3DMODEL_DIR}/Diode_SMD.3dshapes/D_1206_3216Metric.wrl"
