File: pcb_pga2040/connections.kicad_sch (KiCad schematic)
At the start: 3 parts, among them J201 Conn_01x20_Female, J202 Conn_01x20_Female, J203 Conn_01x20_Female

Commit message: update v1.2 pcb, add comments to PGS version, create v1.2 gerbers
Other:
- title: ZX Spectrum Diagnostics -> ZX Spectrum Diagnostics Board PGA2040
Changed lines of the file:
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@@
   (paper "A4")
   (title_block
-    (title "ZX Spectrum Diagnostics")
-    (date "2023-11-30")
+    (title "ZX Spectrum Diagnostics Board PGA2040")
+    (date "2024-03-12")
     (rev "1.1")
   )
